Commit message: feat: add deterministic Nav2 loopback fixture
Add a hardware-independent Nav2 system fixture with explicit TF ownership,
a static obstacle map, NavFn A* planning, regulated pure pursuit control,
and launch-level assertions for goal completion and collision clearance.

File: src/amr_description/urdf/amr.urdf.xacro (robot description, xacro)
@@ -79,3 +79,9 @@
     <origin xyz="-0.18 0 -0.085"/>
   </joint>
+  <link name="base_scan"/>
+  <joint name="base_scan_joint" type="fixed">
+    <parent link="base_link"/>
+    <child link="base_scan"/>
+    <origin xyz="0.18 0 0.10"/>
+  </joint>
 </robot>
